Commit message: mid360 仿真点云时间戳改为帧内相对时间；量程增至 70m
- 每点 timestamp 原为「绝对仿真时间 + CSV 行号」，下游 LIO 无法用于去畸变，
  且导致帧 end_time 漂移；现归一化为点在单帧扫描内的相对时间 [s]
  （CSV 时间列为采样序号，采样率 = 帧点数 × 更新率）
- laser_max_range 5.0 → 70.0（Mid-360 实际量程），室内建图需要更远量程

File: src/robot_scene/xacro/mid360.xacro (robot description, xacro)
@@ -3,5 +3,5 @@
   <xacro:property name="M_PI" value="3.1415926"/>
   <xacro:property name="laser_min_range" value="0.1"/>
-  <xacro:property name="laser_max_range" value="5.0"/>
+  <xacro:property name="laser_max_range" value="70.0"/>
   <xacro:property name="point_rate" value="200000"/>
   <xacro:property name="update_rate" value="10"/>

Commit message: mid360 mesh 路径补 file:// 前缀
裸绝对路径 Gazebo 可解析但 RViz resource_retriever 不认，
导致 RobotModel 显示时 livox 网格加载失败

File: src/robot_scene/xacro/mid360.xacro (robot description, xacro)
@@ -27,5 +27,5 @@
         <origin xyz="0 0 -0.045" rpy="0 0 0"/>
         <geometry>
-          <mesh filename="$(find mid360_simulation)/meshes/livox_frame.STL"/>
+          <mesh filename="file://$(find mid360_simulation)/meshes/livox_frame.STL"/>
         </geometry>
         <material name="livox_dark_grey">
@@ -36,5 +36,5 @@
         <origin xyz="-0.011 -0.02329 -0.005" rpy="0 0 0"/>
         <geometry>
-          <mesh filename="$(find mid360_simulation)/meshes/livox_frame.STL"/>
+          <mesh filename="file://$(find mid360_simulation)/meshes/livox_frame.STL"/>
         </geometry>
       </collision>
